File: PCB/Auckland-LED-Train-Map.kicad_pcb (KiCad board)
At the start: 2 copper layers, 327.8 x 69.9 mm, 212 parts, among them U1 SK6615CS5, U3 Connector, USB-TYPE-C-16P, U4 ESP32-C3FH4, X1 40MHz, 15pF

Commit message: Long Version Checkpoint
Parts:
- removed C15, C16: 15pF, PCM_JLCPCB:C_0402
- removed C17: 100nF, PCM_JLCPCB:C_0402
- removed D07, D400, D401, D402, D403, D404: WS2812B, JLCPCB-Kicad-Footprints:LED-SMD_4P-L1.6-W1.5_XL-1615RGBC-WS2812B
- removed the D105 at (210.0, 14.2)
- removed the D106 at (212.2, 12.0)
- removed the D107 at (213.0, 9.00)
- removed the D202 at (213.0, 6.00)
- removed the D203 at (135.0, -12.0)
- removed the D206 at (134.2, -21.0)
- removed D217, D218, D45, D46, D48, D49, D58, D62, D8, D9: WS2812B, PCM_JLCPCB:LED-SMD_4P-L1.6-W1.5_XL-1615RGBC-WS2812B
- removed the D301 at (138.0, -24.0)
- removed the D302 at (141.0, -24.0)
- removed the D320 at (165.0, 9.00)
- removed L3, L4: 3.9nH,300mA, PCM_JLCPCB:L_0402
- removed L5, L6: 470nH,3.7A, JLCPCB-Kicad-Footprints:L_1008
- removed RT1: 47kΩ,4050, JLCPCB-Kicad-Footprints:RT_0402
- added C100: 10uF, PCM_JLCPCB:C_0402, F.Cu at (-9.00, 50.5)
- added C101: 220nF, PCM_JLCPCB:C_0402, F.Cu at (-8.00, 50.5)
- added C102: 220nF, PCM_JLCPCB:C_0402, F.Cu at (-7.00, 50.5)
- added C104: 220nF, PCM_JLCPCB:C_0402, F.Cu at (159.4, 54.5)
- added C19: 15pF, PCM_JLCPCB:C_0402, F.Cu at (29.6, 19.0)
- added C20: 15pF, PCM_JLCPCB:C_0402, F.Cu at (28.9, 14.2)
- added C22: 100nF, PCM_JLCPCB:C_0402, F.Cu at (-9.26, 10.6)
- added C23: 10uF, PCM_JLCPCB:C_0402, F.Cu at (-5.40, 41.8)
- added C24: 220nF, PCM_JLCPCB:C_0402, F.Cu at (181.0, 51.1)
- added C25: 220nF, PCM_JLCPCB:C_0402, F.Cu at (180.0, 51.1)
- added C26: 10uF, PCM_JLCPCB:C_0402, F.Cu at (179.0, 51.1)
- added C27: 220nF, PCM_JLCPCB:C_0402, F.Cu at (316.0, 52.4)
- added C28: 220nF, PCM_JLCPCB:C_0402, F.Cu at (315.0, 52.4)
- added C29: 10uF, PCM_JLCPCB:C_0402, F.Cu at (314.0, 52.4)
- added C30: 220nF, PCM_JLCPCB:C_0402, F.Cu at (136.0, 5.50)
- added C31: 220nF, PCM_JLCPCB:C_0402, F.Cu at (135.0, 5.50)
- added C32: 10uF, PCM_JLCPCB:C_0402, F.Cu at (134.0, 5.50)
- added C33: 220nF, PCM_JLCPCB:C_0402, F.Cu at (-5.40, 43.6)
- added C34: 220nF, PCM_JLCPCB:C_0402, F.Cu at (-5.40, 45.5)
- added C35: 1uF, PCM_JLCPCB:C_0402, F.Cu at (22.0, 48.0)
- added C36: 1.5pF, PCM_JLCPCB:C_0402, F.Cu at (23.4, 12.0)
- added C37: 1.5pF, PCM_JLCPCB:C_0402, F.Cu at (23.4, 9.00)
- added D109: WS2812B, PCM_JLCPCB:LED-SMD_4P-L1.6-W1.5_XL-1615RGBC-WS2812B, F.Cu at (36.0, 35.0)
- added D111: WS2812B, PCM_JLCPCB:LED-SMD_4P-L1.6-W1.5_XL-1615RGBC-WS2812B, F.Cu at (39.0, 35.0)
- added D130: WS2812B, PCM_JLCPCB:LED-SMD_4P-L1.6-W1.5_XL-1615RGBC-WS2812B, F.Cu at (93.0, 35.0)
- added D138: WS2812B, PCM_JLCPCB:LED-SMD_4P-L1.6-W1.5_XL-1615RGBC-WS2812B, F.Cu at (131.3, 34.7)
- added D140: WS2812B, PCM_JLCPCB:LED-SMD_4P-L1.6-W1.5_XL-1615RGBC-WS2812B, F.Cu at (133.0, 42.0)
- added D150: WS2812B, PCM_JLCPCB:LED-SMD_4P-L1.6-W1.5_XL-1615RGBC-WS2812B, F.Cu at (163.3, 51.7)
- added D151: WS2812B, PCM_JLCPCB:LED-SMD_4P-L1.6-W1.5_XL-1615RGBC-WS2812B, F.Cu at (165.2, 53.8)
- added D152: WS2812B, PCM_JLCPCB:LED-SMD_4P-L1.6-W1.5_XL-1615RGBC-WS2812B, F.Cu at (167.7, 55.1)
- added D160: WS2812B, PCM_JLCPCB:LED-SMD_4P-L1.6-W1.5_XL-1615RGBC-WS2812B, F.Cu at (186.0, 46.0)
- added D168: WS2812B, PCM_JLCPCB:LED-SMD_4P-L1.6-W1.5_XL-1615RGBC-WS2812B, F.Cu at (207.0, 46.0)
- added D172: WS2812B, PCM_JLCPCB:LED-SMD_4P-L1.6-W1.5_XL-1615RGBC-WS2812B, F.Cu at (219.0, 50.0)
- added D174: WS2812B, PCM_JLCPCB:LED-SMD_4P-L1.6-W1.5_XL-1615RGBC-WS2812B, F.Cu at (222.0, 50.0)
- added D186: WS2812B, PCM_JLCPCB:LED-SMD_4P-L1.6-W1.5_XL-1615RGBC-WS2812B, F.Cu at (258.0, 46.0)
- added D188: WS2812B, PCM_JLCPCB:LED-SMD_4P-L1.6-W1.5_XL-1615RGBC-WS2812B, F.Cu at (258.0, 50.0)
- added D300: WS2812B, PCM_JLCPCB:LED-SMD_4P-L1.6-W1.5_XL-1615RGBC-WS2812B, F.Cu at (136.7, 12.7)
- added D305: WS2812B, PCM_JLCPCB:LED-SMD_4P-L1.6-W1.5_XL-1615RGBC-WS2812B, F.Cu at (131.3, 31.3)
- added D306: WS2812B, PCM_JLCPCB:LED-SMD_4P-L1.6-W1.5_XL-1615RGBC-WS2812B, F.Cu at (112.7, 29.3)
- added D315: WS2812B, PCM_JLCPCB:LED-SMD_4P-L1.6-W1.5_XL-1615RGBC-WS2812B, F.Cu at (117.0, 11.0)
- added D318: WS2812B, PCM_JLCPCB:LED-SMD_4P-L1.6-W1.5_XL-1615RGBC-WS2812B, F.Cu at (126.0, 9.00)
- added D322: WS2812B, PCM_JLCPCB:LED-SMD_4P-L1.6-W1.5_XL-1615RGBC-WS2812B, F.Cu at (144.0, 11.0)
- added D323: WS2812B, PCM_JLCPCB:LED-SMD_4P-L1.6-W1.5_XL-1615RGBC-WS2812B, F.Cu at (147.0, 9.00)
- added D324: WS2812B, PCM_JLCPCB:LED-SMD_4P-L1.6-W1.5_XL-1615RGBC-WS2812B, F.Cu at (150.0, 9.00)
- added D340: WS2812B, PCM_JLCPCB:LED-SMD_4P-L1.6-W1.5_XL-1615RGBC-WS2812B, F.Cu at (171.0, 39.0)
- added D341: WS2812B, PCM_JLCPCB:LED-SMD_4P-L1.6-W1.5_XL-1615RGBC-WS2812B, F.Cu at (171.4, 41.8)
- added D342: WS2812B, PCM_JLCPCB:LED-SMD_4P-L1.6-W1.5_XL-1615RGBC-WS2812B, F.Cu at (172.7, 44.3)
- added D343: WS2812B, PCM_JLCPCB:LED-SMD_4P-L1.6-W1.5_XL-1615RGBC-WS2812B, F.Cu at (217.3, 44.3)
- added D344: WS2812B, PCM_JLCPCB:LED-SMD_4P-L1.6-W1.5_XL-1615RGBC-WS2812B, F.Cu at (218.6, 41.8)
- added D345: WS2812B, PCM_JLCPCB:LED-SMD_4P-L1.6-W1.5_XL-1615RGBC-WS2812B, F.Cu at (219.0, 39.0)
- added J1: Conn_01x06_Socket, Connector_PinHeader_2.54mm:PinHeader_1x06_P2.54mm_Vertical, F.Cu at (3.00, 24.0)
- added L1: 3.9nH,300mA, PCM_JLCPCB:L_0402, F.Cu at (23.3, 10.5)
- added L2: 3.9nH,300mA, PCM_JLCPCB:L_0402, F.Cu at (22.5, 10.5)
- added Q1: HL3415A, PCM_JLCPCB:Q_SOT-23, F.Cu at (28.0, 51.5)
- added Q2: MMBT3904, PCM_JLCPCB:Q_SOT-23, F.Cu at (23.0, 50.5)
- added R17: 10kΩ, PCM_JLCPCB:R_0402, F.Cu at (22.0, 45.1)
- added R18: 1kΩ, PCM_JLCPCB:R_0402, F.Cu at (22.5, 46.5)
- added R19: 5.1kΩ, PCM_JLCPCB:R_0402, F.Cu at (318.1, 54.0)
- added R20: 5.1kΩ, PCM_JLCPCB:R_0402, F.Cu at (318.1, 63.0)
- added R21: 0Ω, PCM_JLCPCB:R_1206, F.Cu at (24.7, 20.4)
- added TP1: NAL-NIMT_LED, Custom_Footprints:TestPoint_Pad_D2.0mm, F.Cu at (-23.5, 9.85)
- added TP2: NAL-NIMT_MCU, Custom_Footprints:TestPoint_Pad_D2.0mm, F.Cu at (-23.5, 13.9)
- added TP3: STRAND-MNK_MCU, Custom_Footprints:TestPoint_Pad_D2.0mm, F.Cu at (-23.5, 17.9)
- added TP4: STRAND-MNK_LED, Custom_Footprints:TestPoint_Pad_D2.0mm, F.Cu at (-23.5, 22.0)
- added TP5: PMOS_Gate, Custom_Footprints:TestPoint_Pad_D2.0mm, B.Cu at (24.5, 52.5)
- added TP6: LED_+5V, Custom_Footprints:TestPoint_Pad_D2.0mm, B.Cu at (24.5, 46.5)
- added TP7: NPN_Gate, Custom_Footprints:TestPoint_Pad_D2.0mm, B.Cu at (24.5, 49.5)
- added U2: ESP32-C3FH4, PCM_JLCPCB:QFN-32-1EP_5x5mm_P0.5mm_EP3.7x3.7mm_ThermalVias, F.Cu at (21.2, 16.2)
- added U5: Connector, USB-TYPE-C-16P, PCM_JLCPCB:TYPE-C-SMD_HX-TYPE-C-16PIN, F.Cu at (322.0, 58.5)
- AE1: footprint Inverted_F_Antenna_2.4Ghz_1.0mmPCB_TI_CC2430DB:Inverted_F_Antenna_2.4Ghz_1.0mmPCB_TI_CC2430DB.pretty -> Custom_Footprints:Inverted_F_Antenna_2.4Ghz_1.0mmPCB_TI_CC2430DB.pretty
- C1: value 4.7uF -> 10uF; footprint PCM_JLCPCB:C_0402 -> PCM_JLCPCB:C_0603
- C10: value 2.7pF -> 100nF
- C105: renamed from C22; value 4.7uF -> 220nF
- C12: value 100nF -> 10nF
- C13: value 1pF -> 1uF
- C14: value 22uF -> 100nF; footprint PCM_JLCPCB:C_0603 -> PCM_JLCPCB:C_0402
- C18: value 4.7uF -> 1uF
- C4: value 1uF -> 10uF
- C5: value 10nF -> 10uF
- C6: value 1uF -> 100nF
- C8: value 4.7uF -> 10uF
- C9: value 4.7pF -> 100nF
- D1: value Red -> MMSZ5227B; footprint PCM_JLCPCB:D_0603 -> PCM_JLCPCB:D_SOD-123
- D153: renamed from D405; footprint JLCPCB-Kicad-Footprints:LED-SMD_4P-L1.6-W1.5_XL-1615RGBC-WS2812B -> PCM_JLCPCB:LED-SMD_4P-L1.6-W1.5_XL-1615RGBC-WS2812B
- D154: renamed from D406; footprint JLCPCB-Kicad-Footprints:LED-SMD_4P-L1.6-W1.5_XL-1615RGBC-WS2812B -> PCM_JLCPCB:LED-SMD_4P-L1.6-W1.5_XL-1615RGBC-WS2812B
- D155: renamed from D407; footprint JLCPCB-Kicad-Footprints:LED-SMD_4P-L1.6-W1.5_XL-1615RGBC-WS2812B -> PCM_JLCPCB:LED-SMD_4P-L1.6-W1.5_XL-1615RGBC-WS2812B
- D2: value WS2812B -> Red; footprint PCM_JLCPCB:LED-SMD_4P-L1.6-W1.5_XL-1615RGBC-WS2812B -> PCM_JLCPCB:D_0603
- D3: value WS2812B -> SRV05-4A; footprint PCM_JLCPCB:LED-SMD_4P-L1.6-W1.5_XL-1615RGBC-WS2812B -> PCM_JLCPCB:SOT-23-6_L2.9-W1.6-P0.95-LS2.9-BL
- D307, D319, D321: footprint JLCPCB-Kicad-Footprints:LED-SMD_4P-L1.6-W1.5_XL-1615RGBC-WS2812B -> PCM_JLCPCB:LED-SMD_4P-L1.6-W1.5_XL-1615RGBC-WS2812B
- D320: renamed from D300; footprint JLCPCB-Kicad-Footprints:LED-SMD_4P-L1.6-W1.5_XL-1615RGBC-WS2812B -> PCM_JLCPCB:LED-SMD_4P-L1.6-W1.5_XL-1615RGBC-WS2812B
- D325: renamed from D303; footprint JLCPCB-Kicad-Footprints:LED-SMD_4P-L1.6-W1.5_XL-1615RGBC-WS2812B -> PCM_JLCPCB:LED-SMD_4P-L1.6-W1.5_XL-1615RGBC-WS2812B
- D326: renamed from D304; footprint JLCPCB-Kicad-Footprints:LED-SMD_4P-L1.6-W1.5_XL-1615RGBC-WS2812B -> PCM_JLCPCB:LED-SMD_4P-L1.6-W1.5_XL-1615RGBC-WS2812B
- D327: renamed from D305; footprint JLCPCB-Kicad-Footprints:LED-SMD_4P-L1.6-W1.5_XL-1615RGBC-WS2812B -> PCM_JLCPCB:LED-SMD_4P-L1.6-W1.5_XL-1615RGBC-WS2812B
- D328: renamed from D306; footprint JLCPCB-Kicad-Footprints:LED-SMD_4P-L1.6-W1.5_XL-1615RGBC-WS2812B -> PCM_JLCPCB:LED-SMD_4P-L1.6-W1.5_XL-1615RGBC-WS2812B
- D329: renamed from D308; footprint JLCPCB-Kicad-Footprints:LED-SMD_4P-L1.6-W1.5_XL-1615RGBC-WS2812B -> PCM_JLCPCB:LED-SMD_4P-L1.6-W1.5_XL-1615RGBC-WS2812B
- D330: renamed from D309; footprint JLCPCB-Kicad-Footprints:LED-SMD_4P-L1.6-W1.5_XL-1615RGBC-WS2812B -> PCM_JLCPCB:LED-SMD_4P-L1.6-W1.5_XL-1615RGBC-WS2812B
- D331: renamed from D310; footprint JLCPCB-Kicad-Footprints:LED-SMD_4P-L1.6-W1.5_XL-1615RGBC-WS2812B -> PCM_JLCPCB:LED-SMD_4P-L1.6-W1.5_XL-1615RGBC-WS2812B
- D332: renamed from D311; footprint JLCPCB-Kicad-Footprints:LED-SMD_4P-L1.6-W1.5_XL-1615RGBC-WS2812B -> PCM_JLCPCB:LED-SMD_4P-L1.6-W1.5_XL-1615RGBC-WS2812B
- D333: renamed from D312; footprint JLCPCB-Kicad-Footprints:LED-SMD_4P-L1.6-W1.5_XL-1615RGBC-WS2812B -> PCM_JLCPCB:LED-SMD_4P-L1.6-W1.5_XL-1615RGBC-WS2812B
- D334: renamed from D313; footprint JLCPCB-Kicad-Footprints:LED-SMD_4P-L1.6-W1.5_XL-1615RGBC-WS2812B -> PCM_JLCPCB:LED-SMD_4P-L1.6-W1.5_XL-1615RGBC-WS2812B
- D335: renamed from D314; footprint JLCPCB-Kicad-Footprints:LED-SMD_4P-L1.6-W1.5_XL-1615RGBC-WS2812B -> PCM_JLCPCB:LED-SMD_4P-L1.6-W1.5_XL-1615RGBC-WS2812B
- D336: renamed from D315; footprint JLCPCB-Kicad-Footprints:LED-SMD_4P-L1.6-W1.5_XL-1615RGBC-WS2812B -> PCM_JLCPCB:LED-SMD_4P-L1.6-W1.5_XL-1615RGBC-WS2812B
- D337: renamed from D316; footprint JLCPCB-Kicad-Footprints:LED-SMD_4P-L1.6-W1.5_XL-1615RGBC-WS2812B -> PCM_JLCPCB:LED-SMD_4P-L1.6-W1.5_XL-1615RGBC-WS2812B
- D338: renamed from D317; footprint JLCPCB-Kicad-Footprints:LED-SMD_4P-L1.6-W1.5_XL-1615RGBC-WS2812B -> PCM_JLCPCB:LED-SMD_4P-L1.6-W1.5_XL-1615RGBC-WS2812B
- D339: renamed from D318; footprint JLCPCB-Kicad-Footprints:LED-SMD_4P-L1.6-W1.5_XL-1615RGBC-WS2812B -> PCM_JLCPCB:LED-SMD_4P-L1.6-W1.5_XL-1615RGBC-WS2812B
- D4, D5: value WS2812B -> MM1W5V6; footprint PCM_JLCPCB:LED-SMD_4P-L1.6-W1.5_XL-1615RGBC-WS2812B -> PCM_JLCPCB:D_SOD-123
- D6, D7: value WS2812B -> SS54; footprint PCM_JLCPCB:LED-SMD_4P-L1.6-W1.5_XL-1615RGBC-WS2812B -> PCM_JLCPCB:D_SMA
- F1: value 1.5A -> Polyfuse; footprint JLCPCB-Kicad-Footprints:F_1206 -> Fuse:Fuse_0805_2012Metric_Pad1.15x1.40mm_HandSolder
- R1: value 510Ω -> 10kΩ
- R10: value 47kΩ -> 100Ω
- R11: value 1kΩ -> 0Ω
- R12: value 68kΩ -> 3.3kΩ
- R13: value 15kΩ -> 5.1kΩ
- R15: value 5.1kΩ -> 100Ω
- R16: value 3.3kΩ -> 100kΩ
- R3: value 0Ω -> 10kΩ
- R4: value 0Ω -> 100kΩ
- R6: value 100kΩ -> 0Ω
- R7: value 10kΩ -> 750Ω; footprint PCM_JLCPCB:R_0402 -> PCM_JLCPCB:R_1206
- R8: value 10kΩ -> 0Ω; footprint PCM_JLCPCB:R_0402 -> PCM_JLCPCB:R_1206
- U1: value SK6615CS5 -> XC6206P332MR; footprint JLCPCB-Kicad-Footprints:SOT-23-5_L2.9-W1.6-P0.95-LS2.8-BR -> PCM_JLCPCB:SOT-23-3_L2.9-W1.6-P1.90-LS2.8-BR
- U3: value Connector, USB-TYPE-C-16P -> SN74LVC4245APWR; footprint PCM_JLCPCB:TYPE-C-SMD_HX-TYPE-C-16PIN -> PCM_JLCPCB:TSSOP-24_L7.8-W4.4-P0.65-LS6.4-BL
- U4: value ESP32-C3FH4 -> Connector, USB-TYPE-C-16P; footprint PCM_JLCPCB:QFN-32-1EP_5x5mm_P0.5mm_EP3.7x3.7mm_ThermalVias -> PCM_JLCPCB:TYPE-C-SMD_HX-TYPE-C-16PIN
- moved D207 318.5 mm to (315.0, 50.0), turned to 180 degrees
- moved U3 310.5 mm to (-15.5, 13.0), turned to 0 degrees
- moved R15 302.3 mm to (-9.26, 16.1)
- moved D1 301.4 mm to (-7.30, 27.0)
- moved C4 296.2 mm to (-11.7, 29.9)
- moved C3 295.8 mm to (-11.7, 28.1)
- moved R11 295.8 mm to (-9.26, 14.3)
- moved R10 295.7 mm to (-9.26, 12.4)
- moved R14 292.3 mm to (8.90, 63.0), turned to 90 degrees
- moved C2 290.5 mm to (-11.7, 26.2), turned to 0 degrees
- moved C5 290.0 mm to (-11.7, 31.8), turned to 0 degrees
- moved U1 284.9 mm to (-7.96, 30.8), turned to 0 degrees
- moved R4 283.0 mm to (5.50, 18.4), turned to -90 degrees
- moved U4 281.8 mm to (5.00, 58.5), turned to -90 degrees
- moved C21 281.7 mm to (-9.26, 8.75)
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- renumbered C19 to C103, D10 to D100, D11 to D101, D12 to D102, D13 to D103, D14 to D104, D15 to D105, D16 to D106, D17 to D107, D18 to D108, D19 to D110, D20 to D112, D21 to D113, D22 to D114, D23 to D115, D24 to D116, D25 to D117, D26 to D118, D27 to D119, D28 to D120, D29 to D121, D30 to D122, D31 to D123, D32 to D124, D33 to D125, D34 to D126, D35 to D127, D36 to D128, D37 to D129, D38 to D131, D39 to D132, D40 to D133, D41 to D134, D42 to D135, D43 to D136, D44 to D137, D47 to D139, D51 to D141, D52 to D142, D50 to D143, D53 to D144, D54 to D145, D55 to D146, D56 to D147, D57 to D148, D59 to D149, D60 to D156, D61 to D157, D63 to D158, D64 to D159, D65 to D161, D66 to D162, D67 to D163, D68 to D164, D69 to D165, D70 to D166, D71 to D167, D72 to D169, D73 to D170, D74 to D171, D75 to D173, D76 to D175, D77 to D176, D78 to D177, D79 to D178, D80 to D179, D81 to D180, D82 to D181, D83 to D182, D84 to D183, D85 to D184, D86 to D185, D87 to D187, D88 to D189, D89 to D190, D90 to D191, D91 to D192, D92 to D193, D93 to D194, D94 to D195, D95 to D196, D96 to D197, D97 to D198, D98 to D199, D99 to D200, D100 to D201, D101 to D202, D102 to D203, D103 to D204, D104 to D206, D204 to D301, D202 to D302, D201 to D303, D200 to D304, D216 to D308, D215 to D309, D214 to D310, D213 to D311, D212 to D312, D211 to D313, D210 to D314, D209 to D316, D208 to D317
Connections:
- net Net-(D42-DOUT) renamed NAL-NIMT-2
- net Net-(D68-DOUT) renamed NAL-NIMT-3
- net Net-(D90-DOUT) renamed NAL-NIMT-4
- C10 pad 1: Net-(AE1-A) -> Net-(U2-VDD3P3_CPU)
- C103 pad 1: VBUS -> +5V
- C105 pad 1: VBUS -> +5V
- C11 pad 1: Net-(C11-Pad1) -> Net-(U2-VDD3P3_CPU)
- C12 pad 1: /Reset -> Net-(C12-Pad1)
- C13 pad 1: Net-(AE1-A) -> Net-(C12-Pad1)
- C14 pad 1: +3V3 -> /Reset
- C18 pad 1: VBUS -> VDD_SPI
- C2 pad 1: +3V3 -> VBUS
- C21 pad 1: +3V3 -> VBUS
- C4 pad 1: VDD_SPI -> +3V3
- C7 pad 1: Net-(C11-Pad1) -> Net-(U2-VDD3P3_CPU)
- C8 pad 1: VBUS -> Net-(U2-VDD3P3_CPU)
- C9 pad 1: /Antenna -> Net-(U2-VDD3P3_CPU)
- D1 pad 1: Net-(D1-Pad1) -> +3V3
- D1 pad 2: Net-(D1-Pad2) -> GND
- D100 pad 2: VBUS -> +5V
- D100 pad 4: Net-(D10-DIN) -> NAL-NIMT-1
- D101 pad 2: VBUS -> +5V
- D102 pad 2: VBUS -> +5V
- D103 pad 2: VBUS -> +5V
- D104 pad 2: VBUS -> +5V
- D105 pad 2: VBUS -> +5V
- D106 pad 2: VBUS -> +5V
- D107 pad 2: VBUS -> +5V
- D108 pad 1: Net-(D18-DOUT) -> Net-(D108-DOUT)
- D108 pad 2: VBUS -> +5V
- D110 pad 1: Net-(D19-DOUT) -> Net-(D110-DOUT)
- D110 pad 2: VBUS -> +5V
- D110 pad 4: Net-(D18-DOUT) -> Net-(D109-DOUT)
- D112 pad 2: VBUS -> +5V
- D112 pad 4: Net-(D19-DOUT) -> Net-(D111-DOUT)
- D113 pad 2: VBUS -> +5V
- D114 pad 2: VBUS -> +5V
- D115 pad 2: VBUS -> +5V
- D116 pad 2: VBUS -> +5V
- D117 pad 2: VBUS -> +5V
- D118 pad 2: VBUS -> +5V
- D119 pad 2: VBUS -> +5V
- D120 pad 2: VBUS -> +5V
- D121 pad 2: VBUS -> +5V
- D122 pad 2: VBUS -> +5V
- D123 pad 2: VBUS -> +5V
- D124 pad 2: VBUS -> +5V
- D125 pad 2: VBUS -> +5V
- D126 pad 2: VBUS -> +5V
- D127 pad 2: VBUS -> +5V
- D128 pad 2: VBUS -> +5V
- D129 pad 1: Net-(D37-DOUT) -> Net-(D129-DOUT)
- D129 pad 2: VBUS -> +5V
- D131 pad 2: VBUS -> +5V
- D131 pad 4: Net-(D37-DOUT) -> Net-(D130-DOUT)
- D132 pad 2: VBUS -> +5V
- D133 pad 2: VBUS -> +5V
- D134 pad 2: VBUS -> +5V
- D135 pad 2: VBUS -> +5V
- D136 pad 2: VBUS -> +5V
- D137 pad 2: VBUS -> +5V
- D139 pad 1: Net-(D47-DOUT) -> Net-(D139-DOUT)
- D139 pad 2: VBUS -> +5V
- D139 pad 4: Net-(D46-DOUT) -> Net-(D138-DOUT)
- D141 pad 2: VBUS -> +5V
- D141 pad 4: Net-(D50-DOUT) -> Net-(D140-DOUT)
- D142 pad 1: Net-(D52-DOUT) -> Net-(D142-DOUT)
- D142 pad 2: VBUS -> +5V
- D143 pad 1: Net-(D50-DOUT) -> Net-(D143-DOUT)
- D143 pad 2: VBUS -> +5V
- D143 pad 4: Net-(D49-DOUT) -> Net-(D142-DOUT)
- D144 pad 1: Net-(D53-DOUT) -> Net-(D144-DOUT)
- D144 pad 2: VBUS -> +5V
- D144 pad 4: Net-(D52-DOUT) -> Net-(D143-DOUT)
- D145 pad 1: Net-(D54-DOUT) -> Net-(D145-DOUT)
- D145 pad 2: VBUS -> +5V
- D145 pad 4: Net-(D53-DOUT) -> Net-(D144-DOUT)
- D146 pad 1: Net-(D55-DOUT) -> Net-(D146-DOUT)
- D146 pad 2: VBUS -> +5V
- D146 pad 4: Net-(D54-DOUT) -> Net-(D145-DOUT)
- D147 pad 1: Net-(D56-DOUT) -> Net-(D147-DOUT)
- D147 pad 2: VBUS -> +5V
- D147 pad 4: Net-(D55-DOUT) -> Net-(D146-DOUT)
- D148 pad 1: Net-(D57-DOUT) -> Net-(D148-DOUT)
- D148 pad 2: VBUS -> +5V
- D148 pad 4: Net-(D56-DOUT) -> Net-(D147-DOUT)
- D149 pad 1: Net-(D59-DOUT) -> Net-(D149-DOUT)
- D149 pad 2: VBUS -> +5V
- D149 pad 4: Net-(D58-DOUT) -> Net-(D148-DOUT)
- D153 pad 1: Net-(D57-DOUT) -> Net-(D153-DOUT)
- D153 pad 2: VBUS -> +5V
- D153 pad 4: Net-(D56-DOUT) -> Net-(D152-DOUT)
- D154 pad 1: Net-(D57-DOUT) -> Net-(D154-DOUT)
- D154 pad 2: VBUS -> +5V
- D154 pad 4: Net-(D56-DOUT) -> Net-(D153-DOUT)
- D155 pad 1: Net-(D57-DOUT) -> Onehunga Branch End
- D155 pad 2: VBUS -> +5V
- D155 pad 4: Net-(D56-DOUT) -> Net-(D154-DOUT)
- D156 pad 2: VBUS -> +5V
- D156 pad 4: Net-(D59-DOUT) -> Onehunga Branch End
- D157 pad 1: Net-(D61-DOUT) -> Net-(D157-DOUT)
- D157 pad 2: VBUS -> +5V
- D158 pad 2: VBUS -> +5V
- D158 pad 4: Net-(D62-DOUT) -> Net-(D157-DOUT)
- D159 pad 1: Net-(D64-DOUT) -> Net-(D159-DOUT)
- D159 pad 2: VBUS -> +5V
- D161 pad 2: VBUS -> +5V
- D161 pad 4: Net-(D64-DOUT) -> Net-(D160-DOUT)
- D162 pad 2: VBUS -> +5V
- D163 pad 2: VBUS -> +5V
- D164 pad 2: VBUS -> +5V
- D165 pad 2: VBUS -> +5V
- D166 pad 2: VBUS -> +5V
- D167 pad 1: Net-(D71-DOUT) -> Net-(D167-DOUT)
- D167 pad 2: VBUS -> +5V
- D169 pad 2: VBUS -> +5V
- D169 pad 4: Net-(D71-DOUT) -> Net-(D168-DOUT)
- D170 pad 2: VBUS -> +5V
- D171 pad 1: Net-(D74-DOUT) -> Net-(D171-DOUT)
- D171 pad 2: VBUS -> +5V
- D173 pad 1: Net-(D75-DOUT) -> Net-(D173-DOUT)
- D173 pad 2: VBUS -> +5V
- D173 pad 4: Net-(D74-DOUT) -> Net-(D172-DOUT)
- D175 pad 2: VBUS -> +5V
- D175 pad 4: Net-(D75-DOUT) -> Net-(D174-DOUT)
- D176 pad 2: VBUS -> +5V
- D177 pad 2: VBUS -> +5V
- D178 pad 2: VBUS -> +5V
- D179 pad 2: VBUS -> +5V
- D180 pad 2: VBUS -> +5V
- D181 pad 2: VBUS -> +5V
- D182 pad 2: VBUS -> +5V
- D183 pad 2: VBUS -> +5V
- D184 pad 2: VBUS -> +5V
- D185 pad 1: Net-(D86-DOUT) -> Net-(D185-DOUT)
- D185 pad 2: VBUS -> +5V
- D187 pad 1: Net-(D87-DOUT) -> Net-(D187-DOUT)
- D187 pad 2: VBUS -> +5V
- D187 pad 4: Net-(D86-DOUT) -> Net-(D186-DOUT)
- D189 pad 2: VBUS -> +5V
- D189 pad 4: Net-(D87-DOUT) -> Net-(D188-DOUT)
- D190 pad 2: VBUS -> +5V
- D191 pad 2: VBUS -> +5V
- D192 pad 2: VBUS -> +5V
- D193 pad 2: VBUS -> +5V
- D194 pad 2: VBUS -> +5V
- D195 pad 2: VBUS -> +5V
- D196 pad 2: VBUS -> +5V
- D197 pad 2: VBUS -> +5V
- D198 pad 2: VBUS -> +5V
- D199 pad 2: VBUS -> +5V
- D2 pad 1: Net-(D2-DOUT) -> Net-(D2-Pad1)
- D2 pad 2: VBUS -> Net-(D2-Pad2)
- D200 pad 2: VBUS -> +5V
- D201 pad 2: VBUS -> +5V
- D202 pad 2: VBUS -> +5V
- D203 pad 2: VBUS -> +5V
- D204 pad 1: Net-(D103-DOUT) (its old number) -> Net-(D204-DOUT)
- D204 pad 2: VBUS -> +5V
- D205 pad 2: VBUS -> +5V
- D206 pad 1: unconnected-(D104-DOUT-Pad1) -> Net-(D206-DOUT)
- D206 pad 2: VBUS -> +5V
- D206 pad 4: Net-(D103-DOUT) (its old number) -> Net-(D205-DOUT)
- D207 pad 1: Net-(D207-DOUT) -> unconnected-(D207-DOUT-Pad1)
- D207 pad 2: VBUS -> +5V
- D3 pad 1: Net-(D3-DOUT) -> /D-
- D3 pad 2: VBUS -> GND
- D3 pad 3: GND -> /D+
- D3 pad 4: Net-(D2-DOUT) -> /D+
- D301 pad 1: Net-(D204-DOUT) -> Net-(D301-DOUT)
- D301 pad 2: VBUS -> +5V
- D302 pad 1: Net-(D202-DOUT) (its old number) -> Net-(D302-DOUT)
- D302 pad 2: VBUS -> +5V
- D302 pad 4: Net-(D201-DOUT) (its old number) -> Net-(D301-DOUT)
- D303 pad 1: Net-(D201-DOUT) (its old number) -> Net-(D303-DOUT)
- D303 pad 2: VBUS -> +5V
- D303 pad 4: Net-(D200-DOUT) (its old number) -> Net-(D302-DOUT)
- D304 pad 1: Net-(D200-DOUT) (its old number) -> Net-(D304-DOUT)
- D304 pad 2: VBUS -> +5V
- D304 pad 4: /CRL_Data -> Net-(D303-DOUT)
- D307 pad 1: Net-(D55-DOUT) -> Net-(D307-DOUT)
- D307 pad 2: VBUS -> +5V
- D307 pad 4: Net-(D54-DOUT) -> Net-(D306-DOUT)
- D308 pad 1: Net-(D216-DOUT) -> Net-(D308-DOUT)
- D308 pad 2: VBUS -> +5V
- D308 pad 4: Net-(D215-DOUT) -> Net-(D307-DOUT)
- D309 pad 1: Net-(D215-DOUT) -> Net-(D309-DOUT)
- D309 pad 2: VBUS -> +5V
- D309 pad 4: Net-(D214-DOUT) -> Net-(D308-DOUT)
- D310 pad 1: Net-(D214-DOUT) -> Net-(D310-DOUT)
- D310 pad 2: VBUS -> +5V
- D310 pad 4: Net-(D213-DOUT) -> Net-(D309-DOUT)
- D311 pad 1: Net-(D213-DOUT) -> Net-(D311-DOUT)
- D311 pad 2: VBUS -> +5V
- D311 pad 4: Net-(D212-DOUT) -> Net-(D310-DOUT)
- D312 pad 1: Net-(D212-DOUT) -> Net-(D312-DOUT)
- D312 pad 2: VBUS -> +5V
- D312 pad 4: Net-(D211-DOUT) -> Net-(D311-DOUT)
- D313 pad 1: Net-(D211-DOUT) -> Net-(D313-DOUT)
- D313 pad 2: VBUS -> +5V
- D313 pad 4: Net-(D210-DOUT) -> Net-(D312-DOUT)
- D314 pad 1: Net-(D210-DOUT) -> Net-(D314-DOUT)
- D314 pad 2: VBUS -> +5V
- D314 pad 4: Net-(D209-DOUT) -> Net-(D313-DOUT)
- D316 pad 1: Net-(D209-DOUT) -> Net-(D316-DOUT)
- D316 pad 2: VBUS -> +5V
- D316 pad 4: Net-(D208-DOUT) -> Net-(D315-DOUT)
- D317 pad 1: Net-(D208-DOUT) -> Net-(D317-DOUT)
- D317 pad 2: VBUS -> +5V
- D317 pad 4: Net-(D207-DOUT) -> Net-(D316-DOUT)
- D319 pad 1: Net-(D215-DOUT) -> Net-(D319-DOUT)
- D319 pad 2: VBUS -> +5V
- D319 pad 4: Net-(D214-DOUT) -> Net-(D318-DOUT)
- D320 pad 1: Net-(D47-DOUT) -> Net-(D320-DOUT)
- D320 pad 2: VBUS -> +5V
- D320 pad 4: Net-(D46-DOUT) -> Net-(D319-DOUT)
- D321 pad 1: Net-(D215-DOUT) -> Net-(D321-DOUT)
- D321 pad 2: VBUS -> +5V
- D321 pad 4: Net-(D214-DOUT) -> Net-(D320-DOUT)
- D325 pad 1: Net-(D50-DOUT) -> Net-(D325-DOUT)
- D325 pad 2: VBUS -> +5V
- D325 pad 4: Net-(D49-DOUT) -> Net-(D324-DOUT)
- D326 pad 1: Net-(D50-DOUT) -> Net-(D326-DOUT)
- D326 pad 2: VBUS -> +5V
- D326 pad 4: Net-(D49-DOUT) -> Net-(D325-DOUT)
- D327 pad 1: Net-(D53-DOUT) -> Net-(D327-DOUT)
- D327 pad 2: VBUS -> +5V
- D327 pad 4: Net-(D52-DOUT) -> Net-(D326-DOUT)
- D328 pad 1: Net-(D54-DOUT) -> Net-(D328-DOUT)
- D328 pad 2: VBUS -> +5V
- D328 pad 4: Net-(D53-DOUT) -> Net-(D327-DOUT)
- D329 pad 1: Net-(D56-DOUT) -> Net-(D329-DOUT)
- D329 pad 2: VBUS -> +5V
- D329 pad 4: Net-(D55-DOUT) -> Net-(D328-DOUT)
- D330 pad 1: Net-(D56-DOUT) -> Net-(D330-DOUT)
- D330 pad 2: VBUS -> +5V
- D330 pad 4: Net-(D55-DOUT) -> Net-(D329-DOUT)
- D331 pad 1: Net-(D56-DOUT) -> Net-(D331-DOUT)
- D331 pad 2: VBUS -> +5V
- D331 pad 4: Net-(D55-DOUT) -> Net-(D330-DOUT)
- D332 pad 1: Net-(D213-DOUT) -> Net-(D332-DOUT)
- D332 pad 2: VBUS -> +5V
- D332 pad 4: Net-(D212-DOUT) -> Net-(D331-DOUT)
- D333 pad 1: Net-(D214-DOUT) -> Net-(D333-DOUT)
- D333 pad 2: VBUS -> +5V
- D333 pad 4: Net-(D213-DOUT) -> Net-(D332-DOUT)
- D334 pad 1: Net-(D215-DOUT) -> Net-(D334-DOUT)
- D334 pad 2: VBUS -> +5V
- D334 pad 4: Net-(D214-DOUT) -> Net-(D333-DOUT)
- D335 pad 1: Net-(D213-DOUT) -> Net-(D335-DOUT)
- D335 pad 2: VBUS -> +5V
- D335 pad 4: Net-(D212-DOUT) -> Net-(D334-DOUT)
- D336 pad 1: Net-(D214-DOUT) -> Net-(D336-DOUT)
- D336 pad 2: VBUS -> +5V
- D336 pad 4: Net-(D213-DOUT) -> Net-(D335-DOUT)
- D337 pad 1: Net-(D215-DOUT) -> Net-(D337-DOUT)
- D337 pad 2: VBUS -> +5V
- D337 pad 4: Net-(D214-DOUT) -> Net-(D336-DOUT)
- D338 pad 1: Net-(D213-DOUT) -> Net-(D338-DOUT)
- D338 pad 2: VBUS -> +5V
- D338 pad 4: Net-(D212-DOUT) -> Net-(D337-DOUT)
- D339 pad 1: Net-(D214-DOUT) -> Net-(D339-DOUT)
- D339 pad 2: VBUS -> +5V
- D339 pad 4: Net-(D213-DOUT) -> Net-(D338-DOUT)
- D4 pad 1: Net-(D4-DOUT) -> +5V
- D4 pad 2: VBUS -> GND
- D5 pad 1: Net-(D5-DOUT) -> VBUS
- D5 pad 2: VBUS -> GND
- D6 pad 1: Net-(D6-DOUT) -> Net-(D2-Pad2)
- D6 pad 2: VBUS -> Net-(D6-Pad2)
- D7 pad 1: Net-(D7-DOUT) -> Net-(D2-Pad2)
- D7 pad 2: VBUS -> Net-(D7-Pad2)
- F1 pad 1: Net-(D1-Pad2) -> Net-(D2-Pad2)
- FB1 pad 2: Net-(C11-Pad1) -> Net-(U2-VDD3P3_CPU)
- R1 pad 1: /MCU_TX -> +3V3
- R1 pad 2: Net-(U4-U0TXD) -> /BOOT_IO9
- R10 pad 1: +3V3 -> NAL-NIMT-1
- R10 pad 2: Net-(R10-Pad2) -> Net-(U3-A1)
- R11 pad 1: Net-(R10-Pad2) -> GND
- R11 pad 2: /Temp -> Net-(U3-DIR)
- R12 pad 1: +3V3 -> Net-(D2-Pad1)
- R12 pad 2: Net-(R12-Pad2) -> VBUS
- R13 pad 1: Net-(R12-Pad2) -> Net-(U4-CC1)
- R14 pad 1: Net-(U3-CC1) -> Net-(U4-CC2)
- R15 pad 1: Net-(U3-CC2) -> STRAND-MNK-1
- R15 pad 2: GND -> Net-(U3-A8)
- R16 pad 1: Net-(D1-Pad1) -> VBUS
- R16 pad 2: VBUS -> Net-(Q1-G)
- R2 pad 2: Net-(U4-GPIO2) -> Net-(U2-GPIO8)
- R3 pad 1: /D- -> +3V3
- R3 pad 2: /MCU_D- -> Net-(U2-GPIO2)
- R4 pad 1: /D+ -> +3V3
- R4 pad 2: /MCU_D+ -> /Reset
- R5 pad 1: /MCU_RX -> /D-
- R5 pad 2: Net-(U4-U0RXD) -> /MCU_D-
- R6 pad 1: +3V3 -> /D+
- R6 pad 2: /Reset -> /MCU_D+
- R7 pad 1: +3V3 -> /MCU_TX
- R7 pad 2: Net-(U4-GPIO8) -> Net-(U2-U0TXD)
- R8 pad 1: +3V3 -> Net-(U2-U0RXD)
- R8 pad 2: /BOOT_IO9 -> /MCU_RX
- R9 pad 2: Net-(U4-XTAL_P) -> Net-(U2-XTAL_P)
- U1 pad 1: VBUS -> GND
- U1 pad 2: GND -> +3V3
- U1 pad 3: Net-(U1-SW) -> VBUS
- X1 pad 3: Net-(U4-XTAL_N) -> Net-(U2-XTAL_N)
Routing:
- net +5V: track 0.00 -> 625.9 mm, vias 0 -> 158
- net Net-(D7-Pad2): track 0.00 -> 309.9 mm, vias 0 -> 4
- net Net-(D342-DOUT): track 0.00 -> 47.1 mm, vias 0 -> 2
- net Net-(D6-Pad2): track 0.00 -> 38.8 mm, vias 0 -> 3
- net /D-: track 0.00 -> 31.2 mm, vias 0 -> 2
- net GND: track 135.0 -> 164.1 mm, vias 169 -> 203
- net /D+: track 0.00 -> 26.5 mm, vias 0 -> 2
- net VBUS: track 0.93 -> 27.2 mm, vias 0 -> 2
- net Net-(C12-Pad1): track 0.00 -> 21.0 mm
- net Net-(D305-DOUT): track 0.00 -> 20.7 mm, vias 0 -> 2
- net Net-(U2-VDD3P3_CPU): track 0.00 -> 18.1 mm
- net Onehunga Branch End: track 0.00 -> 15.1 mm, vias 0 -> 2
- net Net-(U4-CC1): track 0.00 -> 9.18 mm
- net Net-(U5-CC1): track 0.00 -> 9.16 mm
- net Net-(D2-Pad2): track 0.00 -> 9.07 mm
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- added copper zone on F.Cu, net Net-(AE1-A)
- removed copper zone on F.Cu, net (none)
- removed copper zone on F.Cu, net +3V3
Other:
- board size 327.8 x 69.9 mm -> 327 x 66 mm
- board text added: "The Strand"

Commit message: PCB Checkpoint
Parts:
- removed C100, C103, C23, C32, C8: 10uF, PCM_JLCPCB:C_0402
- removed C101, C102, C104, C105, C24, C25, C33, C34: 220nF, PCM_JLCPCB:C_0402
- removed the C26 at (179.0, 51.1)
- removed C9: 100nF, PCM_JLCPCB:C_0402
- removed the D339 at (171.0, 36.0)
- removed the D340 at (171.0, 39.0)
- removed FB1: ~, PCM_JLCPCB:FB_0805
- removed R9: 0Ω, PCM_JLCPCB:R_0402
- removed TP3: STRAND-MNK_MCU, Custom_Footprints:TestPoint_Pad_D2.0mm
- added C15: 100nF, PCM_JLCPCB:C_0402, F.Cu at (26.5, 11.5)
- added C29: 10uF, PCM_JLCPCB:C_0402, F.Cu at (119.0, 47.6)
- added C38: 10uF, PCM_JLCPCB:C_0402, F.Cu at (15.3, 50.0)
- added C39: 220nF, PCM_JLCPCB:C_0402, F.Cu at (15.3, 51.0)
- added C40: 220nF, PCM_JLCPCB:C_0402, F.Cu at (15.3, 52.0)
- added C41: 10uF, PCM_JLCPCB:C_0402, F.Cu at (65.7, 25.0)
- added C42: 220nF, PCM_JLCPCB:C_0402, F.Cu at (65.7, 24.0)
- added C43: 220nF, PCM_JLCPCB:C_0402, F.Cu at (65.7, 23.0)
- added L3: 3.9nH,300mA, PCM_JLCPCB:L_0402, F.Cu at (24.0, 11.0)
- added L4: 3.9nH,300mA, PCM_JLCPCB:L_0402, F.Cu at (24.0, 12.0)
- added L5: 15nH,300mA, PCM_JLCPCB:L_0402, F.Cu at (32.5, 15.5)
- added TP8: STRAND-MNK_MCU, Custom_Footprints:TestPoint_Pad_D2.0mm, B.Cu at (9.00, 21.0)
- C7: value 10uF -> 1uF
- TP1, TP2, TP4: moved to B.Cu
- moved D6 216.0 mm to (233.0, 54.0)
- moved D7 216.0 mm to (237.0, 54.0)
- moved F1 216.0 mm to (233.0, 48.5)
- moved D2 216.0 mm to (235.0, 48.5)
- moved R12 216.0 mm to (235.0, 45.8)
- moved D5 215.0 mm to (232.0, 43.0)
- moved C35 212.6 mm to (234.5, 40.5)
- moved D4 212.6 mm to (239.8, 39.0)
- moved Q1 212.6 mm to (240.5, 44.0)
- moved Q2 212.6 mm to (235.5, 43.0)
- moved R16 212.6 mm to (238.0, 43.5)
- moved R18 212.6 mm to (235.0, 39.0)
- moved TP5 212.6 mm to (237.0, 45.0)
- moved TP6 212.6 mm to (237.0, 39.0)
- moved TP7 212.6 mm to (237.0, 42.0)
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- renumbered C29 to C26, D341 to D339, D342 to D340, D343 to D341, D344 to D342, D345 to D343
Connections:
- D339 pad 4: Net-(D340-DOUT) (its old number) -> Net-(D338-DOUT)
- R15 pad 2: Net-(U3-A8) -> Net-(U3-A5)
- U3 pad 10: Net-(U3-A8) -> unconnected-(U3-A8-Pad10)
- U3 pad 14: /STRAND-MNK_MCU -> unconnected-(U3-B8-Pad14)
- U3 pad 17: unconnected-(U3-B5-Pad17) -> /STRAND-MNK_MCU
- U3 pad 7: unconnected-(U3-A5-Pad7) -> Net-(U3-A5)
Routing:
- net Net-(D7-Pad2): track 309.9 -> 11.7 mm, vias 4 -> 2
- net VBUS: track 27.2 -> 278.0 mm, vias 2 -> 3
- net Net-(D6-Pad2): track 38.8 -> 260.3 mm, vias 3 -> 5
- net +5V: track 625.9 -> 574.7 mm, vias 158 -> 165
- net Net-(D305-DOUT): track 20.7 -> 0.96 mm, vias 2 -> 1
- net GND: track 164.1 -> 180.8 mm, vias 203 -> 215
- net /STRAND-MNK_MCU: track 0.00 -> 10.6 mm, vias 0 -> 2
- net /NAL-NIMT_MCU: track 2.94 -> 12.6 mm, vias 0 -> 2
- net Net-(D320-DOUT): track 7.87 -> 0.00 mm
- net Net-(D319-DOUT): track 6.60 -> 0.00 mm, vias 2 -> 0
- net +3V3: track 1.44 -> 6.99 mm
- net /D+: track 26.5 -> 31.6 mm
- net Net-(D307-DOUT): track 1.89 -> 6.82 mm, vias 0 -> 2
- net /Reset: track 3.91 -> 7.29 mm
- net Net-(D134-DOUT): track 7.87 -> 4.87 mm
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Other:
- board size 327 x 66 mm -> 249 x 66 mm
- board text added: "(lib_symbols (symbol "PCM_JLCPCB-Capacitors:0402,10uF" (pin_numbers (hide yes) ) (pin_names (offset 0) ) (exclude_from_sim no) (in_bom yes) (on_board yes) (property "Reference" "C" (at 2.032 1.668 0) (effects (font (size 1.27 1.27)) (justify left) ) ) (property "Value" "10uF" (at 2.032 -0.3782 0) (effects (font (size 0.8 0.8)) (justify left) ) ) (property "Footprint" "PCM_JLCPCB:C_0402" (at -1.77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"

Commit message: - Remove JLCPCB Outputs - V1 RC1
Parts:
- removed R21, R8: 0Ω, PCM_JLCPCB:R_1206
- added C16: 100nF, PCM_JLCPCB:C_0402, F.Cu at (25.9, 20.5)
- added C8: 10uF, PCM_JLCPCB:C_0402, F.Cu at (21.6, 11.5)
- added D8: Green, PCM_JLCPCB:D_0805, F.Cu at (207.0, 15.0)
- added D9: Green, PCM_JLCPCB:D_0805, F.Cu at (207.0, 19.0)
- added R22: 47kΩ, PCM_JLCPCB:R_0402, F.Cu at (204.5, 19.0)
- added R9: 47kΩ, PCM_JLCPCB:R_0402, F.Cu at (204.5, 15.0)
- added S1: Tactile Button, 160gf, PCM_JLCPCB:SW-SMD_4P-L5.1-W5.1-P3.70-LS6.5-TL-2, F.Cu at (207.0, 24.0)
- added S2: Tactile Button, 160gf, PCM_JLCPCB:SW-SMD_4P-L5.1-W5.1-P3.70-LS6.5-TL-2, F.Cu at (207.0, 30.0)
- added S3: Tactile Button, 160gf, PCM_JLCPCB:SW-SMD_4P-L5.1-W5.1-P3.70-LS6.5-TL-2, F.Cu at (207.0, 36.0)
- R7: value 750Ω -> 510Ω; footprint PCM_JLCPCB:R_1206 -> PCM_JLCPCB:R_0402
- moved R2 189.6 mm to (212.5, 22.1), turned to 180 degrees
- moved D1 24.2 mm to (3.10, 31.6), turned to -90 degrees
- moved R7 4.03 mm to (34.5, 23.5)
- moved C20 1.45 mm to (36.3, 14.2)
- moved L5 1.45 mm to (34.0, 15.5)
- moved X1 1.45 mm to (36.6, 16.6)
- moved C19 1.45 mm to (37.0, 19.0)
- moved R3 0.96 mm to (22.1, 12.9)
- moved C18 0.90 mm to (26.8, 20.5)
- moved R11 0.80 mm to (8.00, 12.7)
- moved R10 0.60 mm to (8.00, 13.9)
- moved C10 0.30 mm to (22.7, 15.5)
Connections:
- net Net-(U2-GPIO8) renamed /MODE_BUTTON
- C10 pad 1: Net-(U2-VDD3P3_CPU) -> +3V3
- C11 pad 1: Net-(U2-VDD3P3_CPU) -> +3V3
- C12 pad 1: Net-(C12-Pad1) -> +3V3
- C13 pad 1: Net-(C12-Pad1) -> +3V3
- C15 pad 1: Net-(U2-VDD3P3_CPU) -> Net-(C15-Pad1)
- C7 pad 1: Net-(U2-VDD3P3_CPU) -> Net-(C15-Pad1)
- L3 pad 2: Net-(U2-VDD3P3_CPU) -> Net-(C15-Pad1)
- L4 pad 2: Net-(U2-VDD3P3_CPU) -> Net-(C15-Pad1)
- U2 pad 10: unconnected-(U2-MTDI-Pad10) -> /STRAND-MNK_MCU
- U2 pad 11: Net-(U2-VDD3P3_CPU) -> +3V3
- U2 pad 12: unconnected-(U2-MTCK-Pad12) -> /-BRIGHTNESS_BUTTON
- U2 pad 13: unconnected-(U2-MTDO-Pad13) -> /+BRIGHTNESS_BUTTON
- U2 pad 16: unconnected-(U2-GPIO10-Pad16) -> /WIFI_LED
- U2 pad 17: Net-(U2-VDD3P3_CPU) -> +3V3
- U2 pad 2: Net-(U2-VDD3P3_CPU) -> Net-(C15-Pad1)
- U2 pad 27: Net-(U2-U0RXD) -> /MCU_RX
- U2 pad 3: Net-(U2-VDD3P3_CPU) -> Net-(C15-Pad1)
- U2 pad 31: Net-(C12-Pad1) -> +3V3
- U2 pad 32: Net-(C12-Pad1) -> +3V3
- U2 pad 8: /NAL-NIMT_MCU -> /LVL_Shifter_EN_Active_Low
- U2 pad 9: unconnected-(U2-MTMS-Pad9) -> /NAL-NIMT_MCU
Routing:
- net +3V3: track 6.99 -> 323.6 mm, vias 0 -> 12
- net /-BRIGHTNESS_BUTTON: track 0.00 -> 235.9 mm, vias 0 -> 5
- net /+BRIGHTNESS_BUTTON: track 0.00 -> 228.5 mm, vias 0 -> 5
- net /MODE_BUTTON: track 0.00 -> 222.9 mm, vias 0 -> 5
- net /WIFI_LED: track 0.00 -> 208.7 mm, vias 0 -> 4
- net +5V: track 574.7 -> 695.5 mm, vias 165 -> 163
- net STRAND-MNK-1: track 2.62 -> 102.8 mm, vias 1 -> 6
- net /MCU_RX: track 0.00 -> 47.2 mm, vias 0 -> 6
- net /MCU_D-: track 10.7 -> 53.1 mm
- net /MCU_D+: track 11.6 -> 53.9 mm
- net VBUS: track 278.0 -> 316.5 mm, vias 3 -> 4
- net /MCU_TX: track 0.00 -> 34.7 mm, vias 0 -> 4
- net GND: track 180.8 -> 213.9 mm, vias 215 -> 242
- net /Reset: track 7.29 -> 32.0 mm, vias 0 -> 2
- net NAL-NIMT-1: track 1.82 -> 24.3 mm, vias 1 -> 8
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Other:
- rule solder_mask_min_width: 0.13 -> 0.05
- board text added: "Manungawhau"
- board text added: "Mode"
- board text added: "Power"
- board text added: "Waitematā"
- board text added: "WiFi"
- board text removed: "(lib_symbols (symbol "PCM_JLCPCB-Capacitors:0402,10uF" (pin_numbers (hide yes) ) (pin_names (offset 0) ) (exclude_from_sim no) (in_bom yes) (on_board yes) (property "Reference" "C" (at 2.032 1.668 0) (effects (font (size 1.27 1.27)) (justify left) ) ) (property "Value" "10uF" (at 2.032 -0.3782 0) (effects (font (size 0.8 0.8)) (justify left) ) ) (property "Footprint" "PCM_JLCPCB:C_0402" (at -1.77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"
- board text removed: "Manungawhau (Mt Eden)"
- board text removed: "Waitematā (Britomart)"

Commit message: - V1 RC2 - Add icons
Parts:
- added C9: 10uF, PCM_JLCPCB:C_0402, F.Cu at (34.0, 12.0)
- added D10: Red, PCM_JLCPCB:D_0805, F.Cu at (229.5, 44.0)
- added D11: Red, PCM_JLCPCB:D_0805, F.Cu at (229.5, 38.0)
- added D12: Green, PCM_JLCPCB:D_0805, F.Cu at (229.5, 40.0)
- added G***: LOGO, Custom_Footprints:Brightness_7, F.Cu at (237.0, 39.0)
- added G***: LOGO, Custom_Footprints:Brightness_0, F.Cu at (237.0, 45.0)
- added G***: LOGO, Custom_Footprints:WiFi_Config, F.Cu at (225.0, 39.0)
- added G***: LOGO, Custom_Footprints:Mode_Off_ON, F.Cu at (237.0, 33.0)
- added G***: LOGO, Custom_Footprints:Power, F.Cu at (225.0, 33.0)
- added G***: LOGO, Custom_Footprints:WiFi, F.Cu at (225.0, 45.0)
- added R21: 15kΩ, PCM_JLCPCB:R_0402, F.Cu at (232.0, 38.0)
- added R23: 47kΩ, PCM_JLCPCB:R_0402, F.Cu at (232.0, 40.0)
- added R8: 15kΩ, PCM_JLCPCB:R_0402, F.Cu at (232.0, 44.0)
- D2: footprint PCM_JLCPCB:D_0603 -> PCM_JLCPCB:D_0805
- R12: value 3.3kΩ -> 15kΩ
- moved R2 189.4 mm to (23.2, 17.6), turned to 45 degrees
- moved R22 38.5 mm to (232.0, 46.0), turned to -90 degrees
- moved S1 37.1 mm to (243.0, 33.0)
- moved S2 37.1 mm to (243.0, 39.0)
- moved S3 37.1 mm to (243.0, 45.0)
- moved D9 35.1 mm to (229.5, 46.0), turned to 180 degrees
- moved R9 33.4 mm to (232.0, 34.0), turned to -90 degrees
- moved D8 29.4 mm to (229.5, 34.0), turned to 180 degrees
- moved R18 17.7 mm to (222.0, 51.1)
- moved C35 17.7 mm to (221.5, 52.5)
- moved D4 17.7 mm to (226.8, 51.0)
- moved D5 17.7 mm to (219.0, 55.0)
- moved Q1 17.7 mm to (227.5, 56.0)
- moved Q2 17.7 mm to (222.5, 55.0)
- moved R16 17.7 mm to (225.0, 55.5)
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Connections:
- J1 pad 4: /BOOT_IO9 -> /BOOT_IO9_BUTTON
- R1 pad 2: /BOOT_IO9 -> /BOOT_IO9_BUTTON
- R10 pad 2: Net-(U3-A1) -> Net-(U3-A2)
- R15 pad 2: Net-(U3-A5) -> Net-(U3-A1)
- R2 pad 2: /MODE_BUTTON -> Net-(U2-GPIO8)
- S1 pad 1: /MODE_BUTTON -> /BOOT_IO9_BUTTON
- S1 pad 2: /MODE_BUTTON -> /BOOT_IO9_BUTTON
- U2 pad 10: /STRAND-MNK_MCU -> /CONFIG_LED
- U2 pad 14: /MODE_BUTTON -> Net-(U2-GPIO8)
- U2 pad 15: /BOOT_IO9 -> /BOOT_IO9_BUTTON
- U2 pad 4: unconnected-(U2-GPIO0/XTAL_32K_P-Pad4) -> /LVL_Shifter_EN_Active_Low
- U2 pad 5: unconnected-(U2-GPIO1/XTAL_32K_N-Pad5) -> /STRAND-MNK_MCU
- U2 pad 8: /LVL_Shifter_EN_Active_Low -> /NAL-NIMT_MCU
- U2 pad 9: /NAL-NIMT_MCU -> /LED_+5V_EN_Active_High
- U3 pad 10: unconnected-(U3-A8-Pad10) -> GND
- U3 pad 14: unconnected-(U3-B8-Pad14) -> GND
- U3 pad 15: unconnected-(U3-B7-Pad15) -> GND
- U3 pad 16: unconnected-(U3-B6-Pad16) -> GND
- U3 pad 17: /STRAND-MNK_MCU -> GND
- U3 pad 18: unconnected-(U3-B4-Pad18) -> GND
- U3 pad 19: unconnected-(U3-B3-Pad19) -> GND
- U3 pad 20: unconnected-(U3-B2-Pad20) -> /NAL-NIMT_MCU
- U3 pad 21: /NAL-NIMT_MCU -> /STRAND-MNK_MCU
- U3 pad 4: unconnected-(U3-A2-Pad4) -> Net-(U3-A2)
- U3 pad 5: unconnected-(U3-A3-Pad5) -> GND
- U3 pad 6: unconnected-(U3-A4-Pad6) -> GND
- U3 pad 7: Net-(U3-A5) -> GND
- U3 pad 8: unconnected-(U3-A6-Pad8) -> GND
- U3 pad 9: unconnected-(U3-A7-Pad9) -> GND
Routing:
- net /BOOT_IO9_BUTTON: track 0.00 -> 296.1 mm, vias 0 -> 9
- net /CONFIG_LED: track 0.00 -> 275.5 mm, vias 0 -> 7
- net /LED_+5V_EN_Active_High: track 0.95 -> 249.6 mm, vias 0 -> 4
- net /MODE_BUTTON: track 222.9 -> 0.00 mm, vias 5 -> 0
- net +5V: track 695.5 -> 906.9 mm, vias 163 -> 166
- net /+BRIGHTNESS_BUTTON: track 228.5 -> 274.6 mm, vias 5 -> 7
- net Net-(D2-Pad2): track 8.57 -> 50.9 mm, vias 0 -> 2
- net /WIFI_LED: track 208.7 -> 250.0 mm, vias 4 -> 5
- net +3V3: track 323.6 -> 360.9 mm, vias 12 -> 15
- net /-BRIGHTNESS_BUTTON: track 235.9 -> 271.0 mm, vias 5 -> 7
- net /BOOT_IO9: track 22.8 -> 0.00 mm, vias 2 -> 0
- net VBUS: track 316.5 -> 334.5 mm, vias 4 -> 6
- net /STRAND-MNK_MCU: track 20.4 -> 13.6 mm, vias 2 -> 1
- net GND: track 213.9 -> 208.2 mm, vias 242 -> 320
- net /MCU_D-: track 53.1 -> 57.4 mm
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- added copper zone on F.Cu, net +5V
Other:
- board text removed: "Mode"
- board text removed: "Power"
- board text removed: "WiFi"
