File: PCB/NAL-NIMT-2.kicad_sch (KiCad schematic)
At the start: 27 parts

Commit message: PCB Checkpoint
Parts:
- removed C103: 10uF, PCM_JLCPCB:C_0402, symbol PCM_JLCPCB-Capacitors:0402,10uF
- removed C104, C105: 220nF, PCM_JLCPCB:C_0402, symbol PCM_JLCPCB-Capacitors:0402,220nF
- added C29: 10uF, PCM_JLCPCB:C_0402, symbol PCM_JLCPCB-Capacitors:0402,10uF
- added C30, C31: 220nF, PCM_JLCPCB:C_0402, symbol PCM_JLCPCB-Capacitors:0402,220nF
Connections:
- net +5V: now also C29.1, C30.1, C31.1
- net GND: now also C29.2, C30.2, C31.2

Commit message: - Add Readme - V1 RC3 PCB - Tidy up Schematic - Add Datasheets
Other:
- company: (none) -> Kea Studios
- title: (none) -> Auckland Train Network Live Map
Changed lines of the file:
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@@
 	(generator_version "9.0")
 	(paper "A4")
+	(title_block
+		(title "Auckland Train Network Live Map")
+		(date "2025-04-26")
+		(rev "1")
+		(company "Kea Studios")
+		(comment 1 "©Chris Dirks")
+		(comment 2 "MIT License")
+	)
 	(text "Middlemore"
 		(exclude_from_sim no)

Commit message: Final tweaks for V1.0.0
Parts:
- D136, D137, D138, D139, D140, D141, D142, D143, D144, D145, D146, D147, D148, D149, D150, D156, D157, D158, D159, D160, D161, D162, D163, D164: Manufacturer (none) -> XINGLIGHT; Part (none) -> XL-1615RGBC-WS2812B; Process (none) -> SMT
