File: PCB/NAL-NIMT-3.kicad_sch (KiCad schematic)
At the start: 27 parts

Commit message: - Add Readme - V1 RC3 PCB - Tidy up Schematic - Add Datasheets
Other:
- company: (none) -> Kea Studios
- title: (none) -> Auckland Train Network Live Map
Changed lines of the file:
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@@
 	(generator_version "9.0")
 	(paper "A4")
+	(title_block
+		(title "Auckland Train Network Live Map")
+		(date "2025-04-26")
+		(rev "1")
+		(company "Kea Studios")
+		(comment 1 "©Chris Dirks")
+		(comment 2 "MIT License")
+	)
 	(text "Homai"
 		(exclude_from_sim no)

Commit message: Final tweaks for V1.0.0
Parts:
- D165, D166, D167, D168, D169, D170, D171, D172, D173, D174, D175, D176, D177, D178, D179, D180, D181, D182, D183, D184, D185, D186, D187, D188, D189, D190, D191: Manufacturer (none) -> XINGLIGHT; Part (none) -> XL-1615RGBC-WS2812B; Process (none) -> SMT
