File: PCB/NAL-NIMT-4.kicad_sch (KiCad schematic)
At the start: 16 parts

Commit message: PCB Checkpoint
Parts:
- added C26: 10uF, PCM_JLCPCB:C_0402, symbol PCM_JLCPCB-Capacitors:0402,10uF
- added C27, C28: 220nF, PCM_JLCPCB:C_0402, symbol PCM_JLCPCB-Capacitors:0402,220nF
Connections:
- net +5V: now also C26.1, C27.1, C28.1
- net GND: now also C26.2, C27.2, C28.2

Commit message: - Add Readme - V1 RC3 PCB - Tidy up Schematic - Add Datasheets
Other:
- company: (none) -> Kea Studios
- title: (none) -> Auckland Train Network Live Map
Changed lines of the file:
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@@
 	(generator_version "9.0")
 	(paper "A4")
+	(title_block
+		(title "Auckland Train Network Live Map")
+		(date "2025-04-26")
+		(rev "1")
+		(company "Kea Studios")
+		(comment 1 "©Chris Dirks")
+		(comment 2 "MIT License")
+	)
 	(text "Paerātā"
 		(exclude_from_sim no)

Commit message: Final tweaks for V1.0.0
Parts:
- D192, D193, D194, D195, D196, D197, D198, D199, D200, D201, D202, D203, D204, D205, D206, D207: Manufacturer (none) -> XINGLIGHT; Part (none) -> XL-1615RGBC-WS2812B; Process (none) -> SMT
