File: PCB/Onehunga Branch.kicad_sch (KiCad schematic)
At the start: 5 parts

Commit message: V1.1.0 PCB
Parts:
- D152, D153, D154, D155, D156: value WS2812B -> XL-1615RGBC-WS2812B-S; LCSC C5349954 -> C41413180; Manufacturer XINGLIGHT -> (none); Part XL-1615RGBC-WS2812B -> (none); Process SMT -> (none)
Changed lines of the file:
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@@
 	(title_block
 		(title "Auckland Train Network Live Map")
-		(date "2025-04-26")
-		(rev "1")
+		(date "2025-06-23")
+		(rev "1.1.0")
 		(company "Kea Studios")
 		(comment 1 "©Chris Dirks")
@@
 			)
 		)
-		(property "Value" "WS2812B"
+		(property "Value" "XL-1615RGBC-WS2812B-S"
 			(at 104.3176 21.5777 0)
 			(effects
@@
 					(size 1.27 1.27)
 				)
+				(hide yes)
 			)
 		)
@@
 			)
 		)
-		(property "LCSC" "C5349954"
+		(property "LCSC" "C41413180"
 			(at 93.98 25.4 0)
 			(effects
@@
 			)
 		)
-		(property "Part" "XL-1615RGBC-WS2812B"
+		(property "Circuits" ""
 			(at 93.98 25.4 0)
 			(effects
@@
 			)
 		)
-		(property "Manufacturer" "XINGLIGHT"
+		(property "Current Rating" ""
 			(at 93.98 25.4 0)
 			(effects
@@
 			)
 		)
-		(property "PartID" ""
+		(property "DC Resistance" ""
 			(at 93.98 25.4 0)
 			(effects
@@
 					(size 1.27 1.27)
 				)
-			)
-		)
-		(property "Process" "SMT"
+				(hide yes)
+			)
+		)
+		(property "Impedance @ Frequency" ""
 			(at 93.98 25.4 0)
 			(effects
@@
 					(size 1.27 1.27)
 				)
+				(hide yes)
 			)
 		)
@@
 			)
 		)
-		(property "Value" "WS2812B"
+		(property "Value" "XL-1615RGBC-WS2812B-S"
 			(at 58.5976 21.5777 0)
 			(effects
@@
 					(size 1.27 1.27)
 				)
+				(hide yes)
 			)
 		)
@@
 			)
 		)
-		(property "LCSC" "C5349954"
+		(property "LCSC" "C41413180"
 			(at 48.26 25.4 0)
 			(effects
@@
 			)
 		)
-		(property "Part" "XL-1615RGBC-WS2812B"
+		(property "Circuits" ""
 			(at 48.26 25.4 0)
 			(effects
@@
 			)
 		)
-		(property "Manufacturer" "XINGLIGHT"
+		(property "Current Rating" ""
 			(at 48.26 25.4 0)
 			(effects
@@
 			)
 		)
-		(property "PartID" ""
+		(property "DC Resistance" ""
 			(at 48.26 25.4 0)
 			(effects
@@
 					(size 1.27 1.27)
 				)
-			)
-		)
-		(property "Process" "SMT"
+				(hide yes)
+			)
+		)
+		(property "Impedance @ Frequency" ""
 			(at 48.26 25.4 0)
 			(effects
@@
 					(size 1.27 1.27)
 				)
+				(hide yes)
 			)
 		)
@@
 			)
 		)
-		(property "Value" "WS2812B"
+		(property "Value" "XL-1615RGBC-WS2812B-S"
 			(at 150.0376 21.5777 0)
 			(effects
@@
 					(size 1.27 1.27)
 				)
+				(hide yes)
 			)
 		)
@@
 			)
 		)
-		(property "LCSC" "C5349954"
+		(property "LCSC" "C41413180"
 			(at 139.7 25.4 0)
 			(effects
@@
 			)
 		)
-		(property "Part" "XL-1615RGBC-WS2812B"
+		(property "Circuits" ""
 			(at 139.7 25.4 0)
 			(effects
@@
 			)
 		)
-		(property "Manufacturer" "XINGLIGHT"
+		(property "Current Rating" ""
 			(at 139.7 25.4 0)
 			(effects
@@
 			)
 		)
-		(property "PartID" ""
+		(property "DC Resistance" ""
 			(at 139.7 25.4 0)
 			(effects
@@
 					(size 1.27 1.27)
 				)
-			)
-		)
-		(property "Process" "SMT"
+				(hide yes)
+			)
+		)
+		(property "Impedance @ Frequency" ""
 			(at 139.7 25.4 0)
 			(effects
@@
 					(size 1.27 1.27)
 				)
+				(hide yes)
 			)
 		)
@@
 			)
 		)
-		(property "Value" "WS2812B"
+		(property "Value" "XL-1615RGBC-WS2812B-S"
 			(at 81.4576 21.5777 0)
 			(effects
@@
 					(size 1.27 1.27)
 				)
+				(hide yes)
 			)
 		)
@@
 			)
 		)
-		(property "LCSC" "C5349954"
+		(property "LCSC" "C41413180"
 			(at 71.12 25.4 0)
 			(effects
@@
 			)
 		)
-		(property "Part" "XL-1615RGBC-WS2812B"
+		(property "Circuits" ""
 			(at 71.12 25.4 0)
 			(effects
@@
 			)
 		)
-		(property "Manufacturer" "XINGLIGHT"
+		(property "Current Rating" ""
 			(at 71.12 25.4 0)
 			(effects
@@
 			)
 		)
-		(property "PartID" ""
+		(property "DC Resistance" ""
 			(at 71.12 25.4 0)
 			(effects
@@
 					(size 1.27 1.27)
 				)
-			)
-		)
-		(property "Process" "SMT"
+				(hide yes)
+			)
+		)
+		(property "Impedance @ Frequency" ""
 			(at 71.12 25.4 0)
 			(effects
@@
 					(size 1.27 1.27)
 				)
+				(hide yes)
 			)
 		)
@@
 			)
 		)
-		(property "Value" "WS2812B"
+		(property "Value" "XL-1615RGBC-WS2812B-S"
 			(at 127.1776 21.5777 0)
 			(effects
@@
 					(size 1.27 1.27)
 				)
+				(hide yes)
 			)
 		)
@@
 			)
 		)
-		(property "LCSC" "C5349954"
+		(property "LCSC" "C41413180"
 			(at 116.84 25.4 0)
 			(effects
@@
 			)
 		)
-		(property "Part" "XL-1615RGBC-WS2812B"
+		(property "Circuits" ""
 			(at 116.84 25.4 0)
 			(effects
@@
 			)
 		)
-		(property "Manufacturer" "XINGLIGHT"
+		(property "Current Rating" ""
 			(at 116.84 25.4 0)
 			(effects
@@
 			)
 		)
-		(property "PartID" ""
+		(property "DC Resistance" ""
 			(at 116.84 25.4 0)
 			(effects
@@
 					(size 1.27 1.27)
 				)
-			)
-		)
-		(property "Process" "SMT"
+				(hide yes)
+			)
+		)
+		(property "Impedance @ Frequency" ""
 			(at 116.84 25.4 0)
 			(effects
@@
 					(size 1.27 1.27)
 				)
-			)
-		)
+				(hide yes)
+			)
+		)

Commit message: Update to meet OSHWA Certification
Parts:
- D152, D153, D154, D155, D156: Manufacturer (none) -> XINGLIGHT; Part (none) -> XL-1615RGBC-WS2812B-S
Changed lines of the file:
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@@
+			)
+		)
+		(property "Manufacturer" "XINGLIGHT"
+			(at 93.98 25.4 0)
+			(effects
+				(font
+					(size 1.27 1.27)
+				)
+				(hide yes)
+			)
+		)
+		(property "Part" "XL-1615RGBC-WS2812B-S"
+			(at 93.98 25.4 0)
+			(effects
+				(font
+					(size 1.27 1.27)
+				)
+				(hide yes)
 			)
 		)
@@
 			)
 		)
+		(property "Manufacturer" "XINGLIGHT"
+			(at 48.26 25.4 0)
+			(effects
+				(font
+					(size 1.27 1.27)
+				)
+				(hide yes)
+			)
+		)
+		(property "Part" "XL-1615RGBC-WS2812B-S"
+			(at 48.26 25.4 0)
+			(effects
+				(font
+					(size 1.27 1.27)
+				)
+				(hide yes)
+			)
+		)
 		(pin "2"
 		)
@@
 			)
 		)
+		(property "Manufacturer" "XINGLIGHT"
+			(at 139.7 25.4 0)
+			(effects
+				(font
+					(size 1.27 1.27)
+				)
+				(hide yes)
+			)
+		)
+		(property "Part" "XL-1615RGBC-WS2812B-S"
+			(at 139.7 25.4 0)
+			(effects
+				(font
+					(size 1.27 1.27)
+				)
+				(hide yes)
+			)
+		)
 		(pin "2"
 		)
@@
 			)
 		)
+		(property "Manufacturer" "XINGLIGHT"
+			(at 71.12 25.4 0)
+			(effects
+				(font
+					(size 1.27 1.27)
+				)
+				(hide yes)
+			)
+		)
+		(property "Part" "XL-1615RGBC-WS2812B-S"
+			(at 71.12 25.4 0)
+			(effects
+				(font
+					(size 1.27 1.27)
+				)
+				(hide yes)
+			)
+		)
 		(pin "2"
 		)
@@
 			(at 116.84 25.4 0)
 			(effects
+				(font
+					(size 1.27 1.27)
+				)
+				(hide yes)
+			)
+		)
+		(property "Manufacturer" "XINGLIGHT"
+			(at 116.84 25.4 0)
+			(effects
+				(font
+					(size 1.27 1.27)
+				)
+				(hide yes)
+			)
+		)
+		(property "Part" "XL-1615RGBC-WS2812B-S"
+			(at 116.84 25.4 0)
+			(effects

Commit message: V1.1.1
Other:
- title: Auckland Train Network Live Map -> Auckland Live Train Map
Changed lines of the file:
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@@
 	(paper "A4")
 	(title_block
-		(title "Auckland Train Network Live Map")
-		(date "2025-06-23")
-		(rev "1.1.0")
+		(title "Auckland Live Train Map")
+		(date "2025-07-03")
+		(rev "1.1.1")
 		(company "Kea Studios")
 		(comment 1 "©Chris Dirks")
-		(comment 2 "MIT License")
+		(comment 2 "GPL-3.0-or-later License")
 	)
 	(text "Te Papapa"
