File: PCB/STRAND-MNK-2.kicad_sch (KiCad schematic)
At the start: 4 parts

Commit message: PCB Checkpoint
Parts:
- renumbered D342 to D340, D343 to D341, D344 to D342, D345 to D343
Changed lines of the file:
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@@
 		(dnp no)
 		(fields_autoplaced yes)
-		(property "Reference" "D344"
+		(property "Reference" "D342"
 			(at 134.7976 21.6934 0)
 			(effects
@@
 			(project "Auckland-LED-Train-Map"
 				(path "/ab288f7d-a01b-40d1-8b79-fa22fb371f45/73a3a625-5e65-4151-a327-626a93127f88/e16470c1-e6de-4b7a-8c2a-2890c425ddf6"
-					(reference "D344")
+					(reference "D342")
 					(unit 1)
 				)
@@
 		(dnp no)
 		(fields_autoplaced yes)
-		(property "Reference" "D345"
+		(property "Reference" "D343"
 			(at 157.6576 21.6934 0)
 			(effects
@@
 			(project "Auckland-LED-Train-Map"
 				(path "/ab288f7d-a01b-40d1-8b79-fa22fb371f45/73a3a625-5e65-4151-a327-626a93127f88/e16470c1-e6de-4b7a-8c2a-2890c425ddf6"
-					(reference "D345")
+					(reference "D343")
 					(unit 1)
 				)
@@
 		(dnp no)
 		(fields_autoplaced yes)
-		(property "Reference" "D343"
+		(property "Reference" "D341"
 			(at 111.9376 21.6934 0)
 			(effects
@@
 			(project "Auckland-LED-Train-Map"
 				(path "/ab288f7d-a01b-40d1-8b79-fa22fb371f45/73a3a625-5e65-4151-a327-626a93127f88/e16470c1-e6de-4b7a-8c2a-2890c425ddf6"
-					(reference "D343")
+					(reference "D341")
 					(unit 1)
 				)
@@
 		(dnp no)
 		(fields_autoplaced yes)
-		(property "Reference" "D342"
+		(property "Reference" "D340"
 			(at 50.9776 21.6934 0)
 			(effects
@@
 			(project "Auckland-LED-Train-Map"
 				(path "/ab288f7d-a01b-40d1-8b79-fa22fb371f45/73a3a625-5e65-4151-a327-626a93127f88/e16470c1-e6de-4b7a-8c2a-2890c425ddf6"
-					(reference "D342")
-					(unit 1)
-				)
+					(reference "D340")
+					(unit 1)
+				)

Commit message: - Add Readme - V1 RC3 PCB - Tidy up Schematic - Add Datasheets
Other:
- company: (none) -> Kea Studios
- title: (none) -> Auckland Train Network Live Map
Changed lines of the file:
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@@
 	(generator_version "9.0")
 	(paper "A4")
+	(title_block
+		(title "Auckland Train Network Live Map")
+		(date "2025-04-26")
+		(rev "1")
+		(company "Kea Studios")
+		(comment 1 "©Chris Dirks")
+		(comment 2 "MIT License")
+	)
 	(text "Manukau"
 		(exclude_from_sim no)

Commit message: Final tweaks for V1.0.0
Parts:
- D340, D341, D342, D343: Manufacturer (none) -> XINGLIGHT; Part (none) -> XL-1615RGBC-WS2812B; Process (none) -> SMT
Changed lines of the file:
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@@
+			)
+		)
+		(property "Part" "XL-1615RGBC-WS2812B"
+			(at 124.46 27.94 0)
+			(effects
+				(font
+					(size 1.27 1.27)
+				)
+				(hide yes)
+			)
+		)
+		(property "Manufacturer" "XINGLIGHT"
+			(at 124.46 27.94 0)
+			(effects
+				(font
+					(size 1.27 1.27)
+				)
+				(hide yes)
+			)
+		)
+		(property "PartID" ""
+			(at 124.46 27.94 0)
+			(effects
+				(font
+					(size 1.27 1.27)
+				)
+			)
+		)
+		(property "Process" "SMT"
+			(at 124.46 27.94 0)
+			(effects
+				(font
+					(size 1.27 1.27)
+				)
 			)
 		)
@@
 			)
 		)
+		(property "Part" "XL-1615RGBC-WS2812B"
+			(at 147.32 27.94 0)
+			(effects
+				(font
+					(size 1.27 1.27)
+				)
+				(hide yes)
+			)
+		)
+		(property "Manufacturer" "XINGLIGHT"
+			(at 147.32 27.94 0)
+			(effects
+				(font
+					(size 1.27 1.27)
+				)
+				(hide yes)
+			)
+		)
+		(property "PartID" ""
+			(at 147.32 27.94 0)
+			(effects
+				(font
+					(size 1.27 1.27)
+				)
+			)
+		)
+		(property "Process" "SMT"
+			(at 147.32 27.94 0)
+			(effects
+				(font
+					(size 1.27 1.27)
+				)
+			)
+		)
 		(pin "2"
 		)
@@
 			)
 		)
+		(property "Part" "XL-1615RGBC-WS2812B"
+			(at 101.6 27.94 0)
+			(effects
+				(font
+					(size 1.27 1.27)
+				)
+				(hide yes)
+			)
+		)
+		(property "Manufacturer" "XINGLIGHT"
+			(at 101.6 27.94 0)
+			(effects
+				(font
+					(size 1.27 1.27)
+				)
+				(hide yes)
+			)
+		)
+		(property "PartID" ""
+			(at 101.6 27.94 0)
+			(effects
+				(font
+					(size 1.27 1.27)
+				)
+			)
+		)
+		(property "Process" "SMT"
+			(at 101.6 27.94 0)
+			(effects
+				(font
+					(size 1.27 1.27)
+				)
+			)
+		)
 		(pin "2"
 		)
@@
 			)
 		)
+		(property "Part" "XL-1615RGBC-WS2812B"
+			(at 40.64 27.94 0)
+			(effects
+				(font
+					(size 1.27 1.27)
+				)
+				(hide yes)
+			)
+		)
+		(property "Manufacturer" "XINGLIGHT"
+			(at 40.64 27.94 0)
+			(effects
+				(font
+					(size 1.27 1.27)
+				)
+				(hide yes)
+			)
+		)
+		(property "PartID" ""
+			(at 40.64 27.94 0)
+			(effects
+				(font
+					(size 1.27 1.27)
+				)
+			)
+		)
+		(property "Process" "SMT"
+			(at 40.64 27.94 0)
+			(effects
+				(font
+					(size 1.27 1.27)
+				)
+			)
+		)
