File: PCB/Auckland-LED-Train-Map.kicad_sch (KiCad schematic)
At the start: 102 parts, among them J1 Prog Connector, Q1 HL3415A, Q2 MMBT3904, U1 XC6206P332MR, U2 ESP32-C3FH4, U3 SN74LVC4245APWR, U4 Connector, USB-TYPE-C-16P, U5 Connector, USB-TYPE-C-16P, X1 40MHz, 15pF

Commit message: Fix U3 Footprint
Parts:
- U3: footprint PCM_JLCPCB:TSSOP-24_L7.8-W4.4-P0.65-LS6.4-BL -> Package_SO:TSSOP-24_4.4x7.8mm_P0.65mm
Changed lines of the file:
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@@
 			)
 		)
-		(property "Footprint" "PCM_JLCPCB:TSSOP-24_L7.8-W4.4-P0.65-LS6.4-BL"
+		(property "Footprint" "Package_SO:TSSOP-24_4.4x7.8mm_P0.65mm"
 			(at 228.6 149.86 0)
 			(effects

Commit message: Auckland-V1.1-PCB (#2)
Parts:
- removed C1, C25: 10uF, PCM_JLCPCB:C_0603, symbol PCM_JLCPCB-Capacitors:0603,10uF
- removed C15, C5: 100uF, PCM_JLCPCB:C_1206, symbol PCM_JLCPCB-Capacitors:1206,100uF
- removed D3: SRV05-4A, PCM_JLCPCB:SOT-23-6_L2.9-W1.6-P0.95-LS2.9-BL, symbol PCM_JLCPCB-Diode-Packages:Package, SRV05-4A_C20615829
- removed H4: ~, PCM_JLCPCB:Hole_Tooling_JLCPCB, symbol PCM_JLCPCB-Manufacturing:Tooling Hole, PCM_JLCPCB, 1.152mm
- removed TP10: VBUS, Custom_Footprints:TestPoint_Pad_D1.0mm, symbol Connector:TestPoint
- removed TP11: GND, Custom_Footprints:TestPoint_Pad_D1.0mm, symbol Connector:TestPoint
- removed TP12: WiFi_LED, Custom_Footprints:TestPoint_Pad_D1.0mm, symbol Connector:TestPoint
- removed TP14: Config_LED, Custom_Footprints:TestPoint_Pad_D1.0mm, symbol Connector:TestPoint
- removed TP5: PMOS_Gate, Custom_Footprints:TestPoint_Pad_D1.0mm, symbol Connector:TestPoint
- removed TP6: ALED_5V, Custom_Footprints:TestPoint_Pad_D1.0mm, symbol Connector:TestPoint
- removed TP7: NPN_Gate, Custom_Footprints:TestPoint_Pad_D1.0mm, symbol Connector:TestPoint
- added C1: 10uF, PCM_JLCPCB:C_CASE-A-3216-18(mm), symbol PCM_JLCPCB-Capacitors:CASE-A-3216-18(mm),10uF
- added C15, C5: 100uF, PCM_JLCPCB:C_CASE-B-3528-21(mm), symbol PCM_JLCPCB-Capacitors:CASE-B-3528-21(mm),100uF
- added C25: 10uF, PCM_JLCPCB:C_0402, symbol PCM_JLCPCB-Capacitors:0402,10uF
- added FB1: ~, PCM_JLCPCB:FB_0603, symbol PCM_JLCPCB-Inductors:Ferrite,0603,(2)
- F1: value Polyfuse, 2.5A -> Polyfuse, 2A; footprint Fuse:Fuse_0805_2012Metric_Pad1.15x1.40mm_HandSolder -> Fuse:Fuse_1206_3216Metric; LCSC C2757931 -> C6165195; Manufacturer BHFUSE -> (none); Part BSMD0805L-200 -> (none)
- R22, R23, R9: value 47kΩ -> 100kΩ; symbol PCM_JLCPCB-Resistors:0402,47kΩ -> PCM_JLCPCB-Resistors:0402,100kΩ; LCSC C25792 -> C25741; Part 0402WGF4702TCE -> 0402WGF1003TCE; Resistance 47kΩ -> 100kΩ; Stock 1134503 -> 4111720
Connections:
- net +3V3: now also C25.1, C5.1
- net +5V: now also C15.1
- net GND: now also C1.2, C15.2, C25.2, C5.2
- net VBUS: now also C1.1
- net at D2.2, D6.1, D7.1: now also FB1.1; no longer F1.1
- new net: F1.1, FB1.2
Other:
- moved on the sheet: D1, F1

Commit message: V1.1.0 PCB
Parts:
- removed C16, C17: 100nF, PCM_JLCPCB:C_0402, symbol PCM_JLCPCB-Capacitors:0402,100nF
- removed C23, C24: C_Small, PCM_JLCPCB:C_0402, symbol Device:C_Small
- removed C25, C4, C8: 10uF, PCM_JLCPCB:C_0402, symbol PCM_JLCPCB-Capacitors:0402,10uF
- removed FB1: ~, PCM_JLCPCB:FB_0603, symbol PCM_JLCPCB-Inductors:Ferrite,0603,(2)
- removed H1, H2, H3: ~, PCM_JLCPCB:Hole_Tooling_JLCPCB, symbol PCM_JLCPCB-Manufacturing:Tooling Hole, PCM_JLCPCB, 1.152mm
- removed R11, R26, R5, R6: 0Ω, PCM_JLCPCB:R_0402, symbol PCM_JLCPCB-Resistors:0402,0Ω
- added C25, C4, C8: 1uF, PCM_JLCPCB:C_0402, symbol PCM_JLCPCB-Capacitors:0402,1uF
- C10, C11, C14, C2, C21, C22, C3, C6: value 100nF -> 1uF; symbol PCM_JLCPCB-Capacitors:0402,100nF -> PCM_JLCPCB-Capacitors:0402,1uF; Capacitance 100nF -> 1uF; LCSC C1525 -> C52923; Part CL05B104KO5NNNC -> CL05A105KA5NQNC; Price 0.004USD -> 0.006USD; Stock 20577604 -> 9606588; Temperature Coefficient X7R -> X5R; Voltage Rated 16V -> 25V
- C12: value 10nF -> 1uF; symbol PCM_JLCPCB-Capacitors:0402,10nF -> PCM_JLCPCB-Capacitors:0402,1uF; Capacitance 10nF -> 1uF; LCSC C15195 -> C52923; Part CL05B103KB5NNNC -> CL05A105KA5NQNC; Price 0.005USD -> 0.006USD; Stock 2162276 -> 9606588; Temperature Coefficient X7R -> X5R; Voltage Rated 50V -> 25V
- C13: Stock 6607844 -> 9606588
- C9: value 10uF -> 1uF; symbol PCM_JLCPCB-Capacitors:0402,10uF -> PCM_JLCPCB-Capacitors:0402,1uF; Capacitance 10uF -> 1uF; LCSC C15525 -> C52923; Part CL05A106MQ5NUNC -> CL05A105KA5NQNC; Price 0.007USD -> 0.006USD; Stock 1595146 -> 9606588; Tolerance ±20% -> ±10%; Voltage Rated 6.3V -> 25V
- R12, R21, R8: value 15kΩ -> 10kΩ; symbol PCM_JLCPCB-Resistors:0402,15kΩ -> PCM_JLCPCB-Resistors:0402,10kΩ; LCSC C25756 -> C25744; Minimum Qty 20 -> 5; Part 0402WGF1502TCE -> 0402WGF1002TCE; Resistance 15kΩ -> 10kΩ; Stock 534593 -> 18633144
- R18: value 1kΩ -> 510Ω; symbol PCM_JLCPCB-Resistors:0402,1kΩ -> PCM_JLCPCB-Resistors:0402,510Ω; Attrition Qty 10 -> 12; LCSC C11702 -> C25123; Part 0402WGF1001TCE -> 0402WGF5100TCE; Resistance 1kΩ -> 510Ω; Stock 8259778 -> 1084943
- R4: value 100kΩ -> 10kΩ; symbol PCM_JLCPCB-Resistors:0402,100kΩ -> PCM_JLCPCB-Resistors:0402,10kΩ; LCSC C25741 -> C25744; Minimum Qty 20 -> 5; Part 0402WGF1003TCE -> 0402WGF1002TCE; Resistance 100kΩ -> 10kΩ; Stock 6150463 -> 18633144
- U4, U5: footprint PCM_JLCPCB:TYPE-C-SMD_HX-TYPE-C-16PIN -> Custom_Footprints:TYPE-C-SMD_HX-TYPE-C-16PIN
Connections:
- net MCU_D+ is gone; now on net D+: U2.26 (GPIO19/USB_D+)
- net MCU_D- is gone; now on net D-: U2.25 (GPIO18/USB_D-)
- net +3V3: now also C25.1, C4.1, C8.1
- net GND: now also U3.2 (DIR), C25.2, C4.2, C8.2
- net Reset: now also U2.7 (CHIP_EN)
- net at D2.2, D6.1, D7.1: now also F1.1
Other:
- moved on the sheet: R1, R2, R3

Commit message: Update to meet OSHWA Certification
Parts:
- F1: Manufacturer (none) -> BORN; Part (none) -> SMD1206-200/06N
Changed lines of the file:
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@@
 					(size 1.27 1.27)
 				)
+				(hide yes)
 			)
 		)
@@
 					(size 1.27 1.27)
 				)
+				(hide yes)
 			)
 		)
@@
 					(size 1.27 1.27)
 				)
+				(hide yes)
 			)
 		)
@@
 			)
 		)
-		(property "Description" ""
+		(property "Description" "6V 2A 100A 4A 1206 Resettable Fuses ROHS"
 			(at 68.58 20.32 0)
 			(effects
@@
 			)
 		)
-		(property "Manufacturer" ""
+		(property "Manufacturer" "BORN"
 			(at 68.58 20.32 90)
 			(effects
@@
 			)
 		)
-		(property "Part" ""
+		(property "Part" "SMD1206-200/06N"
 			(at 68.58 20.32 90)
 			(effects
@@
 					(size 1.27 1.27)
 				)
+				(hide yes)
 			)
 		)

Commit message: V1.1.1
Parts:
- added LOGO1: ~, OSHW_Certification_Mark:OSHW-Certification-Mark-Stacked_8x7mm_SilkMask, symbol OSHW_Certification_Mark:OSHW_Certification_Mark_Stacked_Small
Other:
- title: Auckland Train Network Live Map -> Auckland Live Train Map
- moved on the sheet: R1, R2, R3
