File: PCB/NAL-NIMT-1.kicad_sch (KiCad schematic)
At the start: 39 parts

Commit message: PCB Checkpoint
Parts:
- removed C100: 10uF, PCM_JLCPCB:C_0402, symbol PCM_JLCPCB-Capacitors:0402,10uF
- removed C101, C102: 220nF, PCM_JLCPCB:C_0402, symbol PCM_JLCPCB-Capacitors:0402,220nF
- added C38: 10uF, PCM_JLCPCB:C_0402, symbol PCM_JLCPCB-Capacitors:0402,10uF
- added C39, C40: 220nF, PCM_JLCPCB:C_0402, symbol PCM_JLCPCB-Capacitors:0402,220nF
Connections:
- net +5V: now also C38.1, C39.1, C40.1
- net GND: now also C38.2, C39.2, C40.2

Commit message: - Add Readme - V1 RC3 PCB - Tidy up Schematic - Add Datasheets
Other:
- company: (none) -> Kea Studios
- title: (none) -> Auckland Train Network Live Map
Changed lines of the file:
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@@
 	(generator_version "9.0")
 	(paper "A4")
+	(title_block
+		(title "Auckland Train Network Live Map")
+		(date "2025-04-26")
+		(rev "1")
+		(company "Kea Studios")
+		(comment 1 "©Chris Dirks")
+		(comment 2 "MIT License")
+	)
 	(text "Henderson East (1+2)"
 		(exclude_from_sim no)

Commit message: Final tweaks for V1.0.0
Parts:
- D100, D101, D102, D103, D104, D105, D106, D107, D108, D109, D110, D111, D112, D113, D114, D115, D116, D117, D118, D119, D120, D121, D122, D123, D124, D125, D126, D127, D128, D129, D130, D131, D132, D133, D134, D135: Manufacturer (none) -> XINGLIGHT; Part (none) -> XL-1615RGBC-WS2812B; Process (none) -> SMT

Commit message: V1.1.0 PCB
Parts:
- C38: value 10uF -> 1uF; symbol PCM_JLCPCB-Capacitors:0402,10uF -> PCM_JLCPCB-Capacitors:0402,1uF; Capacitance 10uF -> 1uF; LCSC C15525 -> C52923; Part CL05A106MQ5NUNC -> CL05A105KA5NQNC; Price 0.007USD -> 0.006USD; Stock 1595146 -> 9606588; Tolerance ±20% -> ±10%; Voltage Rated 6.3V -> 25V
- C39, C40: value 220nF -> 1uF; symbol PCM_JLCPCB-Capacitors:0402,220nF -> PCM_JLCPCB-Capacitors:0402,1uF; Capacitance 220nF -> 1uF; LCSC C16772 -> C52923; Part CL05B224KO5NNNC -> CL05A105KA5NQNC; Price 0.008USD -> 0.006USD; Stock 351761 -> 9606588; Temperature Coefficient X7R -> X5R; Voltage Rated 16V -> 25V
- D100, D101, D102, D103, D104, D105, D106, D107, D108, D109, D110, D111, D112, D113, D114, D115, D116, D117, D118, D119, D120, D121, D122, D123, D124, D125, D126, D127, D128, D129, D130, D131, D132, D133, D134, D135: value WS2812B -> XL-1615RGBC-WS2812B-S; LCSC C5349954 -> C41413180; Manufacturer XINGLIGHT -> (none); Part XL-1615RGBC-WS2812B -> (none); Process SMT -> (none)

Commit message: Update to meet OSHWA Certification
Parts:
- D100, D101, D102, D103, D104, D105, D106, D107, D108, D109, D110, D111, D112, D113, D114, D115, D116, D117, D118, D119, D120, D121, D122, D123, D124, D125, D126, D127, D128, D129, D130, D131, D132, D133, D134, D135: Manufacturer (none) -> XINGLIGHT; Part (none) -> XL-1615RGBC-WS2812B-S

Commit message: V1.1.1
Other:
- title: Auckland Train Network Live Map -> Auckland Live Train Map
Changed lines of the file:
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@@
 	(paper "A4")
 	(title_block
-		(title "Auckland Train Network Live Map")
-		(date "2025-06-23")
-		(rev "1.1.0")
+		(title "Auckland Live Train Map")
+		(date "2025-07-03")
+		(rev "1.1.1")
 		(company "Kea Studios")
 		(comment 1 "©Chris Dirks")
-		(comment 2 "MIT License")
+		(comment 2 "GPL-3.0-or-later License")
 	)
 	(text "Henderson East (1+2)"
